File: pcb-left/split-ask_left.sch (KiCad schematic (older format))
At the start: 59 parts, among them J1 MJ-4PP-9, SW1 SW_PUSH, SW10 SW_PUSH, SW11 SW_PUSH, SW12 SW_PUSH, SW13 SW_PUSH, SW14 SW_PUSH, SW15 SW_PUSH, SW16 SW_PUSH, SW17 SW_PUSH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

Commit message: update
Parts:
- added D29: D, kbd:D3_TH_SMD, symbol Device:D
- added SW29: SW_PUSH, Alps_Only:ALPS-1U, symbol kbd:SW_PUSH
- RST1: footprint Keebio-Parts:SW_Tactile_SPST_Angled_MJTP1117 -> kbd:ResetSW_1side
Connections:
- net col4: now also SW29.1
- net row4: now also D29.1 (K)
- new net: D29.2 (A), SW29.2
Changed lines of the file:
@@
 F 0 "RST1" H 5150 5855 50  0000 C CNN
 F 1 "SW_PUSH" H 5150 5764 50  0000 C CNN
-F 2 "Keebio-Parts:SW_Tactile_SPST_Angled_MJTP1117" H 5150 5600 50  0001 C CNN
+F 2 "kbd:ResetSW_1side" H 5150 5600 50  0001 C CNN
 F 3 "" H 5150 5600 50  0000 C CNN
 	1    5150 5600
 	1    0    0    -1
 $EndComp
+$Comp
+L kbd:SW_PUSH SW29
+U 1 1 5D466FF6
+P 8800 4700
+F 0 "SW29" H 8800 4955 50  0000 C CNN
+F 1 "SW_PUSH" H 8800 4864 50  0000 C CNN
+F 2 "Alps_Only:ALPS-1U" H 8800 4700 50  0001 C CNN
+F 3 "" H 8800 4700 50  0000 C CNN
+	1    8800 4700
+	1    0    0    -1
+$EndComp
+$Comp
+L Device:D D29
+U 1 1 5D466FFC
+P 9100 4850
+F 0 "D29" V 9146 4771 50  0000 R CNN
+F 1 "D" V 9055 4771 50  0000 R CNN
+F 2 "kbd:D3_TH_SMD" H 9100 4850 50  0001 C CNN
+F 3 "~" H 9100 4850 50  0001 C CNN
+	1    9100 4850
+	0    -1   -1   0
+$EndComp
+Wire Wire Line
+	8500 3950 8500 4700
+Connection ~ 8500 3950
+Wire Wire Line
+	8250 5000 9100 5000
+Connection ~ 8250 5000
 $EndSCHEMATC
