File: pcb-left/split-ask_left.kicad_pcb (KiCad board)
At the start: 2 copper layers, 63 parts, among them J1 MJ-4PP-9, SW1 SW_PUSH, SW10 SW_PUSH, SW11 SW_PUSH, SW12 SW_PUSH, SW13 SW_PUSH, SW14 SW_PUSH, SW15 SW_PUSH, SW16 SW_PUSH, SW17 SW_PUSH, SW18 SW_PUSH, SW19 SW_PUSH, SW2 SW_PUSH, SW20 SW_PUSH, SW21 SW_PUSH, SW22 SW_PUSH, SW23 SW_PUSH, SW24 SW_PUSH, SW25 SW_PUSH, SW26 SW_PUSH, SW27 SW_PUSH, SW28 SW_PUSH, SW29 SW_PUSH, SW3 SW_PUSH, SW4 SW_PUSH, SW5 SW_PUSH, SW6 SW_PUSH, SW7 SW_PUSH, SW8 SW_PUSH, SW9 SW_PUSH, U1 ProMicro

Commit message: update
Parts:
- removed Ref** (x4): Val**, kbd:HOLE
- removed the SW1 at (26.9, 68.8)
- added RST: SW_PUSH, Keebio-Parts:SW_Tactile_SPST_Angled_MJTP1117, B.Cu at (112.1, 15.7)
- D1, D10, D11, D12, D13, D14, D15, D16, D17, D18, D19, D2, D20, D21, D22, D23, D24, D25, D26, D27, D28, D3, D4, D5, D6, D7, D8, D9: footprint kbd:D3_TH -> kbd:D3_TH_SMD
- J1: footprint kbd:MJ-4PP-9 -> kbd:MJ-4PP-9_1side; moved to B.Cu
- moved D2 302.5 mm to (61.9, 33.3), turned to 90 degrees
- moved D4 300.4 mm to (100.0, 33.3), turned to 90 degrees
- moved D3 297.4 mm to (81.0, 33.3), turned to 90 degrees
- moved D1 297.2 mm to (42.9, 33.3), turned to 90 degrees
- moved D5 293.3 mm to (117.9, 33.3), turned to 90 degrees
- moved D6 290.9 mm to (120.3, 33.3), turned to 90 degrees
- moved D9 281.4 mm to (90.5, 52.4), turned to 90 degrees
- moved D10 279.0 mm to (109.5, 52.4), turned to 90 degrees
- moved D11 277.4 mm to (127.4, 52.4), turned to 90 degrees
- moved D12 275.3 mm to (129.8, 52.4), turned to 90 degrees
- moved D8 272.5 mm to (72.6, 52.4), turned to 90 degrees
- moved D7 270.7 mm to (70.2, 52.4), turned to 90 degrees
- moved D18 265.2 mm to (134.5, 71.4), turned to 90 degrees
- moved D13 262.9 mm to (57.1, 71.4), turned to 90 degrees
- moved D16 258.1 mm to (114.3, 71.4), turned to 90 degrees
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- renumbered SW2 to SW1, SW11 to SW10, SW12 to SW11, SW13 to SW12, SW14 to SW13, SW15 to SW14, SW16 to SW15, SW17 to SW16, SW18 to SW17, SW19 to SW18, SW20 to SW19, SW3 to SW2, SW21 to SW20, SW22 to SW21, SW23 to SW22, SW24 to SW23, SW25 to SW24, SW26 to SW25, SW27 to SW26, SW28 to SW27, SW29 to SW28, SW4 to SW3, SW5 to SW4, SW6 to SW5, SW7 to SW6, SW8 to SW7, SW9 to SW8, SW10 to SW9
Other:
- board outline added: 159.5 x 105 mm

Commit message: update
Parts:
- moved D5 19.0 mm to (98.8, 33.3)
- moved D6 19.0 mm to (101.2, 33.3)
- moved D4 17.9 mm to (82.2, 33.3)
- moved RST1 6.27 mm to (112.1, 21.9)
- moved J1 6.21 mm to (119.1, 19.2)
- moved U1 5.88 mm to (37.5, 52.3)
- moved D3 1.19 mm to (79.8, 33.3)
- renumbered RST to RST1
Other:
- board size 159.5 x 105 mm -> 165.4 x 98.7 mm

Commit message: routing
Routing:
- net row4: track 0.00 -> 183.2 mm
- net col3: track 0.00 -> 181.7 mm
- net col5: track 0.00 -> 150.5 mm
- net row3: track 0.00 -> 147.6 mm
- net col4: track 0.00 -> 141.7 mm
- net col2: track 0.00 -> 134.8 mm
- net GND: track 0.00 -> 131.7 mm
- net row2: track 0.00 -> 126.9 mm
- net col1: track 0.00 -> 125.4 mm
- net row1: track 0.00 -> 115.7 mm
- net data: track 0.00 -> 113.3 mm
- net row0: track 0.00 -> 108.3 mm
- net reset: track 0.00 -> 94.5 mm
- net VCC: track 0.00 -> 92.6 mm
- net col0: track 0.00 -> 90.0 mm
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
Commit message: update
Routing:
- added copper zone on B.Cu, net (none)
- added copper zone on F.Cu, net (none)
Changed lines of the file:
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@@
   )
   (setup
-    (last_trace_width 0.5)
+    (last_trace_width 0.25)
     (user_trace_width 0.5)
     (trace_clearance 0.2)
@@
   (segment (start 149.9 86.4875) (end 149.9 76.9625) (width 0.25) (layer B.Cu) (net 44))
   (segment (start 149.9 76.9625) (end 140.375 67.4375) (width 0.25) (layer B.Cu) (net 44))
+  (zone (net 0) (net_name "") (layer F.Cu) (hatch edge 0.508)
+    (connect_pads (clearance 0.508))
+    (min_thickness 0.254)
+    (fill yes (arc_segments 32) (thermal_gap 0.508) (thermal_bridge_width 0.508))
+    (polygon
+      (pts
+        (xy 15 15) (xy 15 130) (xy 195 130) (xy 195 15)
+      )
+    )
+  )
+  (zone (net 0) (net_name "") (layer B.Cu) (hatch edge 0.508)
+    (connect_pads (clearance 0.508))
+    (min_thickness 0.254)
+    (fill yes (arc_segments 32) (thermal_gap 0.508) (thermal_bridge_width 0.508))
+    (polygon
+      (pts
+        (xy 15 15) (xy 15 130) (xy 195 130) (xy 195 15)
+      )
+    )
+  )
 )

Commit message: update
Parts:
- added D29: D, kbd:D3_TH_SMD, F.Cu at (150.0, 109.5)
- added HOLE1: HOLE, kbd:HOLE, F.Cu at (42.9, 42.1)
- added HOLE2: Val**, kbd:HOLE, F.Cu at (119.1, 42.1)
- added HOLE3: HOLE, kbd:HOLE, F.Cu at (42.9, 100.8)
- added HOLE4: HOLE, kbd:HOLE, F.Cu at (95.2, 100.8)
- added HOLE5: HOLE, kbd:HOLE, F.Cu at (156.4, 100.8)
- added SW29: SW_PUSH, Alps_Only:ALPS-1U, F.Cu at (166.0, 109.6)
- RST1: footprint Keebio-Parts:SW_Tactile_SPST_Angled_MJTP1117 -> kbd:ResetSW_1side
- moved RST1 91.6 mm to (25.7, 52.4), turned to 270 degrees
- moved SW28 25.5 mm to (140.5, 109.5)
- moved U1 20.0 mm to (43.5, 71.4)
- moved D13 17.9 mm to (75.0, 71.4)
- moved D7 17.9 mm to (52.4, 52.4)
- moved J1 4.76 mm to (119.1, 24.0)
- moved D14 1.19 mm to (77.4, 71.4)
- moved D8 1.19 mm to (71.4, 52.4)
Routing:
- net reset: track 94.5 -> 11.8 mm
- net col4: track 141.7 -> 182.3 mm
- net Net-(D29-Pad2): track 0.00 -> 23.6 mm
- net col3: track 181.7 -> 158.3 mm
- net row3: track 147.6 -> 125.9 mm
- net row0: track 108.3 -> 129.7 mm
- net Net-(D13-Pad2): track 18.5 -> 36.9 mm
- net Net-(D7-Pad2): track 34.5 -> 16.1 mm
- net row4: track 183.2 -> 167.6 mm
- net row2: track 126.9 -> 112.0 mm
- net data: track 113.3 -> 126.9 mm
- net row1: track 115.7 -> 128.6 mm
- net col5: track 150.5 -> 157.9 mm
- net GND: track 131.7 -> 135.0 mm
- net col1: track 125.4 -> 122.6 mm
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Other:
- board size 165.4 x 98.7 mm -> 161.7 x 95.2 mm
- board text added: "Split ASK: Left Side / PCB Designed by Ryo Nakae"
