File: pcb-right/split-ask_right.sch (KiCad schematic (older format))
At the start: 59 parts, among them J1 MJ-4PP-9, SW1 SW_PUSH, SW10 SW_PUSH, SW11 SW_PUSH, SW12 SW_PUSH, SW13 SW_PUSH, SW14 SW_PUSH, SW15 SW_PUSH, SW16 SW_PUSH, SW17 SW_PUSH, SW18 SW_PUSH, SW19 SW_PUSH, SW2 SW_PUSH, SW20 SW_PUSH, SW21 SW_PUSH, SW22 SW_PUSH, SW23 SW_PUSH, SW24 SW_PUSH, SW25 SW_PUSH, SW26 SW_PUSH, SW27 SW_PUSH, SW28 SW_PUSH, SW3 SW_PUSH, SW4 SW_PUSH, SW5 SW_PUSH, SW6 SW_PUSH, SW7 SW_PUSH, SW8 SW_PUSH, SW9 SW_PUSH, U1 ProMicro

Commit message: update
Parts:
- added D15, D16, D33, D34, D7, D8: D, kbd:D3_TH_SMD, symbol Device:D
- added SW15, SW16, SW33, SW34, SW7: SW_PUSH, Alps_Only:ALPS-1U, symbol kbd:SW_PUSH
- added SW8: SW_PUSH, Alps_Only:ALPS-1.5U, symbol kbd:SW_PUSH
- SW17: renamed from SW13; footprint Alps_Only:ALPS-1.75U -> Alps_Only:ALPS-1U
- SW23: renamed from SW19; footprint Alps_Only:ALPS-2.25U -> Alps_Only:ALPS-1U
- SW28: renamed from SW24; footprint Alps_Only:ALPS-1U -> Alps_Only:ALPS-2.25U
- SW31: renamed from SW27; footprint Alps_Only:ALPS-1.75U -> Alps_Only:ALPS-1U
- SW9: renamed from SW7; footprint Alps_Only:ALPS-1.5U -> Alps_Only:ALPS-1U
- renumbered D8 to D10, D9 to D11, D10 to D12, D11 to D13, D12 to D14, D13 to D17, D14 to D18, D15 to D19, D16 to D20, D17 to D21, D18 to D22, D19 to D23, D20 to D24, D21 to D25, D22 to D26, D23 to D27, D24 to D28, D25 to D29, D26 to D30, D27 to D31, D28 to D32, D7 to D9, SW8 to SW10, SW9 to SW11, SW10 to SW12, SW11 to SW13, SW12 to SW14, SW14 to SW18, SW15 to SW19, SW16 to SW20, SW17 to SW21, SW18 to SW22, SW20 to SW24, SW21 to SW25, SW22 to SW26, SW23 to SW27, SW25 to SW29, SW26 to SW30, SW28 to SW32
Connections:
- net col4: now also SW33.1
- net col5: now also SW34.1
- net row0: now also D7.1 (K), D8.1 (K)
- net row1: now also D15.1 (K), D16.1 (K)
- net row4: now also D33.1 (K), D34.1 (K)
- net col7: now reaches U1.13 (B6/10)
- net col7: now also SW16.1, SW8.1
- net col6: now reaches U1.14 (B2/16)
- net col6: now also SW15.1, SW7.1
- new net: D7.2 (A), SW7.2
- new net: D8.2 (A), SW8.2
- new net: D15.2 (A), SW15.2
- new net: D16.2 (A), SW16.2
- new net: D33.2 (A), SW33.2
- new net: D34.2 (A), SW34.2
- no-connect marks 8 -> 6

Commit message: update
Parts:
- RST1: footprint Keebio-Parts:SW_Tactile_SPST_Angled_MJTP1117 -> kbd:ResetSW_1side
Changed lines of the file:
@@
 EESchema Schematic File Version 4
+LIBS:split-ask_right-cache
 EELAYER 29 0
 EELAYER END
@@
 F 0 "RST1" H 5150 5855 50  0000 C CNN
 F 1 "SW_PUSH" H 5150 5764 50  0000 C CNN
-F 2 "Keebio-Parts:SW_Tactile_SPST_Angled_MJTP1117" H 5150 5600 50  0001 C CNN
+F 2 "kbd:ResetSW_1side" H 5150 5600 50  0001 C CNN
 F 3 "" H 5150 5600 50  0000 C CNN
 	1    5150 5600
